File: kicadFiles/keebsPCB.sch (KiCad schematic (older format))
At the start: 260 parts, among them J1 USB_C_Receptacle, J2 Conn_01x04_Male, Q1 AO4406AL, SW1 MXSwitch, SW10 MXSwitch, SW11 MXSwitch, SW12 MXSwitch, SW13 MXSwitch, SW14 MXSwitch, SW15 MXSwitch, SW16 MXSwitch, SW17 MXSwitch, SW18 MXSwitch, SW19 MXSwitch, SW2 MXSwitch, SW20 MXSwitch, SW21 MXSwitch, SW22 MXSwitch, SW23 MXSwitch, SW24 MXSwitch, SW25 MXSwitch, SW26 MXSwitch, SW27 MXSwitch, SW28 MXSwitch, SW29 MXSwitch, SW3 MXSwitch, SW30 MXSwitch, SW31 MXSwitch, SW32 MXSwitch, SW33 MXSwitch, SW34 MXSwitch, SW35 MXSwitch, SW36 MXSwitch, SW37 MXSwitch, SW38 MXSwitch, SW39 MXSwitch, SW4 MXSwitch, SW40 MXSwitch, SW41 MXSwitch, SW42 MXSwitch, SW43 MXSwitch, SW44 MXSwitch, SW45 MXSwitch, SW46 MXSwitch, SW47 MXSwitch, SW48 MXSwitch, SW49 MXSwitch, SW5 MXSwitch, SW50 MXSwitch, SW51 MXSwitch, SW6 MXSwitch, SW7 MXSwitch, SW8 MXSwitch, SW9 MXSwitch, U1 STM32F303CCT6, U2 MCP1700-3302E_SOT23, Y1 8MHz

Commit message: [Update] Places switches
Parts:
- removed C1, C2: 22p, Capacitor_SMD:C_0805_2012Metric_Pad1.15x1.40mm_HandSolder, symbol Device:C_Small
- removed C7, C9: 4.7n, Capacitor_SMD:C_0805_2012Metric_Pad1.15x1.40mm_HandSolder, symbol Device:C_Small
- removed CA1, CVBus2, CVBus3: 100n, Capacitor_SMD:C_0805_2012Metric_Pad1.15x1.40mm_HandSolder, symbol Device:C_Small
- removed CVBus4: 1u, Capacitor_SMD:C_0402_1005Metric, symbol Device:C_Small
- removed CVBus5: 4.7u, Capacitor_SMD:C_0805_2012Metric_Pad1.15x1.40mm_HandSolder, symbol Device:C_Small
- removed DF1: RB060M-60TR, acheronComponents:D_SOD-123, symbol Device:D_Schottky_Small
- removed H7: CASE, MountingHole:MountingHole_2.2mm_M2_Pad_Via, symbol Mechanical:MountingHole_Pad
- removed J1: USB_C_Receptacle, USBconnector:TYPE-C-31-M-13, symbol Connector:USB_C_Receptacle
- removed J2: Conn_01x04_Male, acheronConnectors:JSTBM04B-ASRS, symbol Connector:Conn_01x04_Male
- removed L2: LogoBack, sharkLogo:skark, symbol Mechanical:MountingHole
- removed L4: BrazilianFlag, sharkLogo:brazilFlag, symbol Mechanical:MountingHole
- removed L5: usFlag, sharkLogo:usFlag, symbol Mechanical:MountingHole
- removed LED1, LED10, LED11, LED12, LED13, LED14, LED15, LED16, LED17, LED18, LED19, LED2, LED20, LED21, LED22, LED23, LED24, LED25, LED26, LED27, LED28, LED29, LED3, LED30, LED31, LED32, LED33, LED34, LED35, LED36, LED37, LED38, LED39, LED4, LED40, LED41, LED42, LED43, LED44, LED45, LED46, LED47, LED48, LED49, LED5, LED50, LED51, LED6, LED7, LED8, LED9: LED, acheronComponents:thtLED, symbol acheronSymbols:LED
- removed Q1: AO4406AL, acheronComponents:AO4406AL, symbol acheronSymbols:AO4406AL
- removed QRST1: BC847, Package_TO_SOT_SMD:SOT-23, symbol Transistor_BJT:BC847
- removed R5, R6: 1M, Resistor_SMD:R_1206_3216Metric_Pad1.42x1.75mm_HandSolder, symbol Device:R
- removed RA1, RA2, RB1, RB2, RPGate1: 10k, Resistor_SMD:R_1206_3216Metric_Pad1.42x1.75mm_HandSolder, symbol Device:R_Small
- removed RD+1, RD-1: 22R, Resistor_SMD:R_1206_3216Metric_Pad1.42x1.75mm_HandSolder, symbol Device:R_Small
- removed RD+Up1: 1.5k, Resistor_SMD:R_1206_3216Metric_Pad1.42x1.75mm_HandSolder, symbol Device:R_Small
- removed RGB1, RGB2, RGB3, RGB4, RGB5, RGB6, RGB7, RGB8: WS2812B, acheronComponents:LED_WS2812B, symbol LED:WS2812B
- removed RL1, RL10, RL11, RL12, RL13, RL14, RL15, RL16, RL17, RL18, RL19, RL2, RL20, RL21, RL22, RL23, RL24, RL25, RL26, RL27, RL28, RL29, RL3, RL30, RL31, RL32, RL33, RL34, RL35, RL36, RL37, RL38, RL39, RL40, RL41, RL42, RL43, RL44, RL45, RL46, RL47, RL48, RL5, RL6, RL7, RL8, RL9: 360, Resistor_SMD:R_1206_3216Metric, symbol Device:R_Small
- removed RL4: R_LED, Resistor_SMD:R_1206_3216Metric, symbol Device:R_Small
- removed ROT1, ROT2: Rotary_Encoder_Switch, acheronHardware:ALPS_EC11E, symbol Device:Rotary_Encoder_Switch
- removed RSGate1: 100, Resistor_SMD:R_1206_3216Metric_Pad1.42x1.75mm_HandSolder, symbol Device:R_Small
- removed U1: STM32F303CCT6, Package_QFP:LQFP-48_7x7mm_P0.5mm, symbol acheronSymbols:STM32F303CCT6
- removed Y1: 8MHz, acheronComponents:Crystal_SMD_5032-4Pin_5.0x3.2mm, symbol Device:Crystal_GND24
- added CB2: 10n, Capacitor_SMD:C_0402_1005Metric, symbol Device:C_Small
- added CB3, CB8: 100n, Capacitor_SMD:C_0402_1005Metric, symbol Device:C_Small
- added CB4, CB6: 4.7uF, Capacitor_SMD:C_0402_1005Metric, symbol Device:C_Small
- added CB7: 100nF, Capacitor_SMD:C_0402_1005Metric, symbol Device:C_Small
- added CSH1: 4.7nF, Capacitor_SMD:C_0805_2012Metric, symbol Device:C_Small
- added CUSB1: 100n, Capacitor_SMD:C_0805_2012Metric_Pad1.15x1.40mm_HandSolder, symbol Device:C_Small
- added D49, D50, D51, D52, D53, D54, D55, D56, D57, D58, D59, D60, D61: 1N4148, acheron_Components:D_SOD-123, symbol Device:D
- added DF1: RB060M-60TR, acheron_Components:D_SOD-123, symbol Device:D_Schottky
- added H10, H8: Oval Mounting Hole, acheron_MountingHoles:MoutingHole_Oval_BackOnly_7mm_5.0x2.5mm, symbol Mechanical:MountingHole
- added H7, H9: Oval Mounting Hole, acheron_MountingHoles:MoutingHole_Oval_7mm_5.0x2.5mm, symbol Mechanical:MountingHole
- added J1: TYPE-C-31-M12_13, acheron_Connectors:TYPE-C-31-M-12, symbol acheronSymbols:TYPE-C-31-M12_13
- added J5: Conn_01x06_Male, acheron_Connectors:HEADER_6PIN_HORIZONTAL, symbol Connector:Conn_01x06_Male
- added L3: Label, SPV1_graphics:SPV1_preAlpha_Label_15x32mm, symbol Mechanical:MountingHole
- added QRST1: DTC123J, Package_TO_SOT_SMD:SOT-23, symbol Transistor_BJT:DTC123J
- added RSH1: 1M, acheron_Components:R_SMD_1026, symbol Device:R_Small
- added SW52, SW55, SW59, SW61: MXSwitch, acheron_MX:MX100H, symbol acheronSymbols:MXSwitch
- added SW53: MXSwitch, acheron_MX:MX275H, symbol acheronSymbols:MXSwitch
- added SW54, SW56, SW58, SW60: MXSwitch, acheron_MX:MX150H, symbol acheronSymbols:MXSwitch
- added SW57: MXSwitch, acheron_MX:MX700HR, symbol acheronSymbols:MXSwitch
- added U1: STM32F072-LQFP48, acheron_Components:LQFP-48_7x7mm_P0.5mm, symbol acheronSymbols:STM32F072-LQFP48
- added U2: USBLC6-2SC6, acheron_Components:SOT-23-6, symbol Power_Protection:USBLC6-2SC6
- CB1: value 100n -> 1uF; footprint Capacitor_SMD:C_0805_2012Metric_Pad1.15x1.40mm_HandSolder -> Capacitor_SMD:C_0402_1005Metric
- CB5: renamed from CVBus1; footprint Capacitor_SMD:C_0805_2012Metric_Pad1.15x1.40mm_HandSolder -> Capacitor_SMD:C_0402_1005Metric
- CRST1: value 4.7n -> 10u
- D1, D10, D11, D12, D13, D14, D15, D16, D17, D18, D19, D2, D20, D21, D22, D23, D24, D25, D26, D27, D28, D29, D3, D30, D31, D32, D33, D34, D35, D36, D37, D38, D39, D4, D40, D41, D42, D43, D44, D45, D46, D47, D48, D5, D6, D7, D8, D9: footprint acheronComponents:D_SOD-123 -> acheron_Components:D_SOD-123
- DRST1, DS1: footprint Diode_SMD:D_0805_2012Metric_Pad1.15x1.40mm_HandSolder -> acheron_Components:D_SOD-123
- F1: value 1A -> Polyfuse; footprint Fuse:Fuse_0805_2012Metric_Pad1.15x1.40mm_HandSolder -> acheron_Components:Fuse_1812_4532
- H1, H6: value MountingHole -> Half Side Hole; footprint MountingHole:MountingHole_2.5mm_Pad -> acheron_MountingHoles:halfSideHole
- H2: value MountingHole -> Mounting Hole; footprint MountingHole:MountingHole_2.5mm_Pad -> acheron_MountingHoles:MoutingHole_Oval_7mm_5.0x2.5mm
- H3, H5: value MountingHole -> Oval Mounting Hole; footprint MountingHole:MountingHole_2.5mm_Pad -> acheron_MountingHoles:MoutingHole_Oval_BackOnly_7mm_5.0x2.5mm
- H4: value MountingHole -> Oval Mounting Hole; footprint MountingHole:MountingHole_2.5mm_Pad -> acheron_MountingHoles:MoutingHole_Oval_7mm_5.0x2.5mm
- L1: value Logo -> Keebs Logo; footprint sharkLogo:sharkLogo -> keebsLogo:keebsLogo
- L2: renamed from L3; footprint sharkLogo:osh-logo -> oshLogo:osh-logo
- RCC1, RRST1: footprint Resistor_SMD:R_1206_3216Metric_Pad1.42x1.75mm_HandSolder -> acheron_Components:R_SMD_1026
- SW1, SW10, SW11, SW12, SW13, SW16, SW17, SW18, SW19, SW2, SW20, SW21, SW22, SW23, SW24, SW25, SW26, SW27, SW3, SW30, SW31, SW32, SW33, SW34, SW35, SW36, SW37, SW38, SW39, SW4, SW40, SW43, SW44, SW45, SW46, SW47, SW48, SW5, SW6, SW7, SW8, SW9: footprint acheronKeyboardSwitches:MX100 -> acheron_MX:MX100H
- SW14: footprint acheronKeyboardSwitches:MX100 -> acheron_MX:MX200H
- SW15, SW28: footprint acheronKeyboardSwitches:MX100 -> acheron_MX:MX150H
- SW29: footprint acheronKeyboardSwitches:MX100 -> acheron_MX:MX175H
- SW41: footprint acheronKeyboardSwitches:MX100 -> acheron_MX:MX225H
- SW42: footprint acheronKeyboardSwitches:MX100 -> acheron_MX:MX225
- SW49, SW50, SW51: footprint acheronKeyboardSwitches:MX200R -> acheron_MX:MX100H
- SWRST1: footprint smdPushBtn:smdPushBtn -> acheron_Hardware:smdPushBtn
- renumbered CSin1 to CSI1, CSout1 to CSO1, U2 to U3
Connections:
- net 3.3V: now also CB1.2, CB5.2, CB2.2, CB3.2, CB4.2, CB6.2, CB7.1, CB8.2, J5.6 (Pin_6), U1.1 (VBAT), U1.24 (VDD), U1.36 (VDDIO2), U1.48 (VDD), U1.9 (VDDA); no longer CB5.1
- net 5V: now also DF1.1 (K)
- net BOOT0: now also J5.3 (Pin_3), U1.44 (BOOT0)
- net Col1: now also SW15.1 (Col), SW29.1 (Col), SW42.1 (Col), SW54.1 (Col); no longer SW13.1 (Col), SW25.1 (Col), SW37.1 (Col)
- net Col10: now also SW24.1 (Col), SW38.1 (Col), SW51.1 (Col), SW59.1 (Col); no longer SW22.1 (Col), SW34.1 (Col), SW46.1 (Col)
- net Col11: now also SW25.1 (Col), SW39.1 (Col), SW52.1 (Col), SW60.1 (Col); no longer SW23.1 (Col), SW35.1 (Col), SW47.1 (Col)
- net Col12: now also SW26.1 (Col), SW40.1 (Col), SW53.1 (Col); no longer SW24.1 (Col), SW36.1 (Col), SW48.1 (Col)
- net Col2: now also SW16.1 (Col), SW30.1 (Col), SW43.1 (Col), SW55.1 (Col); no longer SW14.1 (Col), SW26.1 (Col), SW38.1 (Col)
- net Col3: now also SW17.1 (Col), SW31.1 (Col), SW44.1 (Col), SW56.1 (Col); no longer SW15.1 (Col), SW27.1 (Col), SW39.1 (Col)
- net Col4: now also SW18.1 (Col), SW32.1 (Col), SW45.1 (Col); no longer SW16.1 (Col), SW28.1 (Col), SW40.1 (Col)
- net Col5: now also SW19.1 (Col), SW33.1 (Col), SW46.1 (Col); no longer SW17.1 (Col), SW29.1 (Col), SW41.1 (Col), SW49.1 (Col)
- net Col6: now also SW20.1 (Col), SW34.1 (Col), SW47.1 (Col); no longer SW18.1 (Col), SW30.1 (Col), SW42.1 (Col), SW50.1 (Col)
- net Col7: now also SW21.1 (Col), SW35.1 (Col), SW48.1 (Col), SW57.1 (Col); no longer SW19.1 (Col), SW31.1 (Col), SW43.1 (Col), SW51.1 (Col)
- net Col8: now also SW22.1 (Col), SW36.1 (Col), SW49.1 (Col); no longer SW20.1 (Col), SW32.1 (Col), SW44.1 (Col)
- net Col9: now also SW23.1 (Col), SW37.1 (Col), SW50.1 (Col), SW58.1 (Col); no longer SW21.1 (Col), SW33.1 (Col), SW45.1 (Col)
- net D+: now also U1.33 (USB_DP/PA12), U2.3 (IO2)
- net D-: now also U1.32 (USB_DM/TIM1_CH4/PA11), U2.1 (IO1)
- net GND: now also CB5.1, CB2.1, CB3.1, CB4.1, CB6.1, CB7.2, CB8.1, CSH1.1, CUSB1.1, DF1.2 (A), J1.A1 (GND), J1.B1 (GND), J5.1 (Pin_1), QRST1.2 (E), RSH1.2, U1.23 (VSS), U1.35 (VSS), U1.47 (VSS), U1.8 (VSSA), U2.2 (GND); no longer CB5.2
- net NRST: now also J5.2 (Pin_2), QRST1.3 (C), U1.7 (NRST)
- net Row1: now also D13.1 (K), D14.1 (K)
- net Row2: now also D25.1 (K), D26.1 (K), D27.1 (K), D28.1 (K); no longer D13.1 (K), D14.1 (K), D15.1 (K)
- net Row3: now also D37.1 (K), D38.1 (K), D39.1 (K), D40.1 (K), D41.1 (K); no longer D25.1 (K), D26.1 (K), D27.1 (K), D28.1 (K)
- net Row4: now also D49.1 (K), D50.1 (K), D51.1 (K), D52.1 (K), D53.1 (K), D61.1 (K); no longer D37.1 (K), D38.1 (K), D39.1 (K), D40.1 (K), D41.1 (K)
- net VBUS: now also CUSB1.2, J1.A4 (VBUS), J1.B4 (VBUS), U2.5 (VBUS)
- net at D41.2 (A), SW41.2 (Row): no longer SW49.2 (Row)
- net at D42.2 (A), SW42.2 (Row): no longer SW50.2 (Row)
- net at D43.2 (A), SW43.2 (Row): no longer SW51.2 (Row)
- net at RCC1.2: now also J1.A5 (CC1), J1.B5 (CC2)
- net at DRST1.2 (A), SWRST1.2: now also QRST1.1 (B)
- net EncS1: no longer names the net of D37.2 (A), SW37.2 (Row)
- net EncS3: no longer names the net of D48.2 (A), SW48.2 (Row)
- new net: D49.2 (A), SW49.2 (Row)
- new net: D50.2 (A), SW50.2 (Row)
- new net: D51.2 (A), SW51.2 (Row)
- new net: D52.2 (A), SW52.2 (Row)
- new net: D53.2 (A), SW53.2 (Row)
- new net: D54.2 (A), SW54.2 (Row)
- new net: D55.2 (A), SW55.2 (Row)
- new net: D56.2 (A), SW56.2 (Row)
- new net: D57.2 (A), SW57.2 (Row)
- new net: D58.2 (A), SW58.2 (Row)
- new net: D59.2 (A), SW59.2 (Row)
- new net: D60.2 (A), SW60.2 (Row)
- new net: D61.2 (A), SW61.2 (Row)
- new net Col13: SW13.1 (Col), SW27.1 (Col), SW41.1 (Col), SW61.1 (Col)
- new net Col14: SW14.1 (Col), SW28.1 (Col)
- new net DBus+: J1.A7 (D-), J1.B7 (D-), U2.4 (IO2)
- new net DBus-: J1.A6 (D+), J1.B6 (D+), U2.6 (IO1)
- new net Row5: D54.1 (K), D55.1 (K), D56.1 (K), D57.1 (K), D58.1 (K), D59.1 (K), D60.1 (K)
- new net SHIELD: CSH1.2, J1.S (SHIELD), RSH1.1
- new net SWCLK: J5.5 (Pin_5), U1.37 (SWCLK/PA14)
- new net SWDIO: J5.4 (Pin_4), U1.34 (SWDIO/PA13)
- no-connect marks 10 -> 2
Other:
- note added: "CBx are the bypass capacitors. Their value is specified in reference [2]."
- note added: "MCU"
- note added: "REFERENCES"
- note added: "Serial programming"
- note added: "Shield"
- note added: "USD ESD"
- note added: "[1] STM32F072x8 / STM32F072xB datasheet"
- note added: "[2] AN4080 Application note"
- note added: "https://www.st.com/content/ccc/resource/technical/document/application_note/c9/19/d7/b8/6b/0e/4c/d3/DM00051986.pdf/files/DM00051986.pdf/jcr:content/translations/en.DM00051986.pdf"
- note added: "https://www.st.com/resource/en/datasheet/stm32f072rb.pdf"
- note removed: "ESD\nProtection"
- note removed: "Encoder nets"
- note removed: "I2C Connector"
- note removed: "MCU and crystal"
- note removed: "Mounting holes"
- note removed: "Polyfuse PPTC RTC"
- note removed: "RGB"
- note removed: "Shield\nnet"
- note removed: "Switch LED matrix"
- note removed: "Switch matrix\n"
- note removed: "Voltage regulation\ncapacitor bank\n"
- moved on the sheet: CB5, CRST1, CRST2, CSI1, CSO1, D1, D10, D11, D12, D13, D2, D3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
