File: kicadFiles/keebsPCB.sch (KiCad schematic (older format))
At the start: 160 parts, among them J1 TYPE-C-31-M12_13, J5 Conn_01x06_Male, SW1 ESC, SW10 9, SW11 0, SW12 -_, SW13 =+, SW14 BKSP_200, SW15 TAB_150, SW16 Q, SW17 W, SW18 E, SW19 R, SW2 1, SW20 T, SW21 Y, SW22 U, SW23 I, SW24 L, SW25 O, SW26 P, SW27 [{, SW28 ]}, SW29 CAPS_175, SW3 2, SW30 A, SW31 S, SW32 D, SW33 F, SW34 G, SW35 H, SW36 J, SW37 K, SW38 L, SW39 :;, SW4 3, SW40 \", SW41 ENTER_225, SW42 LSHIFT_225, SW43 Z, SW44 X, SW45 C, SW46 V, SW47 B, SW48 N, SW49 M, SW5 4, SW50 <,, SW51 .>, SW52 ?/, SW53 RSHIFT_275, SW54 MXSwitch, SW55 MXSwitch, SW56 MXSwitch, SW57 MXSwitch, SW58 MXSwitch, SW59 MXSwitch, SW6 5, SW60 MXSwitch, SW7 6, SW8 7, SW9 8, U1 STM32F072-LQFP48, U2 USBLC6-2SC6, U3 MCP1700-3302E_SOT23

Commit message: Update: finished routing
Parts:
- removed J5: Conn_01x06_Male, acheron_Connectors:HEADER_6PIN_HORIZONTAL, symbol Connector:Conn_01x06_Male
- added J2: Conn_ARM_JTAG_SWD_10, acheron_Connectors:Conn_ARM_JTAG_SWD_10, symbol Connector:Conn_ARM_JTAG_SWD_10
- added J3: Conn_01x14, acheron_Connectors:PinHeader_1x7_P2.54mm_Vertical, symbol Connector_Generic:Conn_01x07
- added J4: Conn_01x14, acheron_Connectors:PinHeader_1x8_P2.54mm_Vertical, symbol Connector_Generic:Conn_01x08
- added RCC2: 5.1k, Resistor_SMD:R_0402_1005Metric, symbol Device:R_Small
- CUSB1: footprint Capacitor_SMD:C_0805_2012Metric_Pad1.15x1.40mm_HandSolder -> Capacitor_SMD:C_0402_1005Metric
- RCC1: footprint acheron_Components:R_SMD_1026 -> Resistor_SMD:R_0402_1005Metric
Connections:
- net Col14 is gone; now on net Col13: SW14.1 (Col), SW28.1 (Col)
- net 3.3V: now also J2.1 (VTref)
- net Col1: now also U1.25 (PB12)
- net Col10: now also SW58.1 (Col), U1.45 (I2C1_SCL/TIM16_CH1/PB8); no longer SW59.1 (Col)
- net Col11: now also SW59.1 (Col), U1.43 (2C1_SDA/PB7); no longer SW60.1 (Col)
- net Col12: now also SW60.1 (Col), U1.42 (I2C1_SCL/PB6)
- net Col13: now also U1.41 (SPI1_MOSI/I2S1_SD/TIM3_CH2/PB5)
- net Col2: now also U1.11 (PA1/ADC_IN1)
- net Col3: now also U1.10 (PA0/ADC_IN0)
- net Col4: now also U1.6 (PF1/OSC_OUT)
- net Col5: now also U1.5 (PF0/OSC_IN)
- net Col6: now also U1.4 (PC15/OSC32_OUT)
- net Col7: now also U1.3 (PC14/OSC32_IN)
- net Col8: now also U1.2 (PC13)
- net Col9: now also U1.46 (SPI2_NSS/I2S2_WS/I2C1_SDA/TIM17_CH1/PB9); no longer SW58.1 (Col)
- net GND: now also J2.3 (GND), J2.5 (GND), J2.9 (GNDDetect), RCC2.1
- net NRST: now also J2.10 (~RESET~)
- net Row1: now also U1.40 (SPI1_MISO/I2S1_MCK/TIM3_CH1/PB4); no longer D14.1 (K)
- net Row2: now also U1.39 (SPI1_SCK/I2S1_CK/TIM2_CH2/PB3); no longer D28.1 (K)
- net Row3: now also U1.12 (PA2/ADC_IN2)
- net Row4: now also D14.1 (K), U1.13 (PA3/TIM15_CH2/ADC_IN3)
- net Row5: now also D28.1 (K), U1.14 (PA4/TIM14_CH1/ADC_IN4)
- net SWCLK: now also J2.4 (SWDCLK/TCK)
- net SWDIO: now also J2.2 (SWDIO/TMS)
- net at J1.A5 (CC1), RCC1.2: no longer J1.B5 (CC2)
- new net: J1.B5 (CC2), RCC2.2
- no-connect marks 2 -> 4
Other:
- moved on the sheet: D14, D28, D58, D59, D60, RCC1, SW14, SW28, SW58, SW59, SW60

Commit message: Update: add label, run DRC
Parts:
- added L3: Keebs Label, keebsLogo:keebsLabel, symbol Mechanical:MountingHole
- added L4: Keebs Label Mask, keebsLogo:keebsLabelMask, symbol Mechanical:MountingHole
Connections:
- net Extra15: now reaches U1.15 (PA5/ADC_IN5/DAC_OUT2)
- net Extra15: now also J4.8 (Pin_8)
- net Extra14: now reaches U1.16 (PA6/ADC_IN6/TIM3_CH1/TIM16_CH1)
- net Extra14: now also J4.7 (Pin_7)
- net Extra13: now reaches U1.17 (PA7/TIM3_CH2/TIM14_CH1/ADC_IN7)
- net Extra13: now also J4.6 (Pin_6)
- net Extra12: now reaches U1.18 (PB0/TIM3_CH3/ADC_IN8)
- net Extra12: now also J4.5 (Pin_5)
- net Extra11: now reaches U1.19 (PB1/TIM3_CH4/TIM14_CH1/ADC_IN9)
- net Extra11: now also J4.4 (Pin_4)
- net Extra10: now reaches U1.20 (PB2)
- net Extra10: now also J4.3 (Pin_3)
- net Extra9: now reaches U1.21 (PB10/SPI2_SCK/I2C2_SCL/TIM2_CH3)
- net Extra9: now also J4.2 (Pin_2)
- net Extra8: now reaches U1.22 (PB11/TIM2_CH4/I2C2_SDA)
- net Extra8: now also J4.1 (Pin_1)
- net Extra7: now reaches U1.26 (SPI2_SCK/I2S2_CK/I2C2_SCL/PB13)
- net Extra7: now also J3.7 (Pin_7)
- net Extra6: now reaches U1.27 (PB14/SPI2_MISO/I2S2_MCK/I2C2_SDA/TIM15_CH1/PB15)
- net Extra6: now also J3.6 (Pin_6)
- net Extra5: now reaches U1.28 (SPI2_MOSI/I2S2_SD/PB15)
- net Extra5: now also J3.5 (Pin_5)
- net Extra4: now reaches U1.29 (TIM1_CH1/PA8)
- net Extra4: now also J3.4 (Pin_4)
- net Extra3: now reaches U1.30 (TIM1_CH2/PA9)
- net Extra3: now also J3.3 (Pin_3)
- net Extra2: now reaches U1.31 (TIM1_CH3/PA10)
- net Extra2: now also J3.2 (Pin_2)
- net Extra1: now reaches U1.38 (PA2)
- net Extra1: now also J3.1 (Pin_1)
Other:
- note added: "SWD"
- note removed: "Serial programming"
- moved on the sheet: J2
Changed lines of the file:
@@
 Wire Wire Line
 	21750 15900 21750 15950
-Text Notes 12725 14650 0    100  Italic 20
-Serial programming
+Text Notes 13300 12075 0    100  Italic 20
+SWD
 $Comp
 L power:GND #PWR0103
 U 1 1 5CFDFC6D
-P 13375 14100
-F 0 "#PWR0103" H 13375 13850 50  0001 C CNN
-F 1 "GND" V 13380 13972 50  0000 R CNN
-F 2 "" H 13375 14100 50  0001 C CNN
-F 3 "" H 13375 14100 50  0001 C CNN
-	1    13375 14100
-	1    0    0    -1
-$EndComp
-Wire Wire Line
-	14050 13425 13975 13425
-Text GLabel 14050 13325 2    50   Input ~ 0
+P 13250 13950
+F 0 "#PWR0103" H 13250 13700 50  0001 C CNN
+F 1 "GND" V 13255 13822 50  0000 R CNN
+F 2 "" H 13250 13950 50  0001 C CNN
+F 3 "" H 13250 13950 50  0001 C CNN
+	1    13250 13950
+	1    0    0    -1
+$EndComp
+Wire Wire Line
+	13925 13275 13850 13275
+Text GLabel 13925 13175 2    50   Input ~ 0
 SWCLK
-Text GLabel 14050 13425 2    50   Input ~ 0
+Text GLabel 13925 13275 2    50   Input ~ 0
 SWDIO
 Wire Wire Line
-	13975 13325 14050 13325
-Wire Wire Line
-	13375 14025 13375 14100
-Text GLabel 13475 12750 1    50   Input ~ 0
+	13850 13175 13925 13175
+Wire Wire Line
+	13250 13875 13250 13950
+Text GLabel 13350 12600 1    50   Input ~ 0
 3.3V
 Wire Wire Line
-	13475 12825 13475 12750
-Wire Wire Line
-	14050 13125 13975 13125
-Text GLabel 14050 13125 2    50   Input ~ 0
+	13350 12675 13350 12600
+Wire Wire Line
+	13925 12975 13850 12975
+Text GLabel 13925 12975 2    50   Input ~ 0
 NRST
 $Comp
@@
 	9100 13950 9100 13900
 Wire Notes Line width 20
-	12525 14450 12525 15925
-Wire Notes Line width 20
-	12525 14450 14425 14450
-Wire Notes Line width 20
-	14425 14450 14425 15925
+	12550 11850 14450 11850
 Wire Notes Line width 20
 	12525 15925 14425 15925
@@
 Shield
 Wire Notes Line width 20
-	12525 14750 14425 14750
+	12550 12150 14450 12150
 Wire Notes Line width 20
 	12650 16500 15200 16500
@@
 	19250 19450 19250 19400
 $Comp
-L Connector:Conn_ARM_JTAG_SWD_10 J2
-U 1 1 5DD65212
-P 13475 13425
-F 0 "J2" H 13032 13471 50  0000 R CNN
-F 1 "Conn_ARM_JTAG_SWD_10" H 13032 13380 50  0000 R CNN
-F 2 "acheron_Connectors:Conn_ARM_JTAG_SWD_10" H 13475 13425 50  0001 C CNN
-F 3 "http://infocenter.arm.com/help/topic/com.arm.doc.ddi0314h/DDI0314H_coresight_components_trm.pdf" V 13125 12175 50  0001 C CNN
-	1    13475 13425
-	1    0    0    -1
-$EndComp
-$Comp
 L power:GND #PWR0114
 U 1 1 5DDA2A9F
-P 13475 14100
-F 0 "#PWR0114" H 13475 13850 50  0001 C CNN
-F 1 "GND" V 13480 13972 50  0000 R CNN
-F 2 "" H 13475 14100 50  0001 C CNN
-F 3 "" H 13475 14100 50  0001 C CNN
-	1    13475 14100
-	1    0    0    -1
-$EndComp
-Wire Wire Line
-	13475 14025 13475 14100
-NoConn ~ 13975 13625
-NoConn ~ 13975 13525
+P 13350 13950
+F 0 "#PWR0114" H 13350 13700 50  0001 C CNN
+F 1 "GND" V 13355 13822 50  0000 R CNN
+F 2 "" H 13350 13950 50  0001 C CNN
+F 3 "" H 13350 13950 50  0001 C CNN
+	1    13350 13950
+	1    0    0    -1
+$EndComp
+Wire Wire Line
+	13350 13875 13350 13950
+NoConn ~ 13850 13475
+NoConn ~ 13850 13375
 $Comp
 L Connector_Generic:Conn_01x07 J3
@@
 	1    0    0    -1
 $EndComp
+Wire Notes Line width 20
+	12550 14500 14450 14500
+$Comp
+L Connector:Conn_ARM_JTAG_SWD_10 J2
+U 1 1 5DD65212
+P 13350 13275
+F 0 "J2" V 12750 13350 50  0000 R CNN
+F 1 "Conn_ARM_JTAG_SWD_10" V 12850 13750 50  0000 R CNN
+F 2 "acheron_Connectors:Conn_ARM_JTAG_SWD_10" H 13350 13275 50  0001 C CNN
+F 3 "http://infocenter.arm.com/help/topic/com.arm.doc.ddi0314h/DDI0314H_coresight_components_trm.pdf" V 13000 12025 50  0001 C CNN
+	1    13350 13275
+	1    0    0    -1
+$EndComp
+Wire Wire Line
+	15625 12925 15700 12925
+Text GLabel 15625 12925 0    50   Input ~ 0
+Extra1
+Wire Notes Line width 20
+	14450 11850 14450 14500
+Wire Notes Line width 20
+	12550 11850 12550 14500
+Wire Wire Line
+	15625 13025 15700 13025
+Text GLabel 15625 13025 0    50   Input ~ 0
+Extra2
+Wire Wire Line
+	15625 13125 15700 13125
+Text GLabel 15625 13125 0    50   Input ~ 0
+Extra3
+Wire Wire Line
+	15625 13225 15700 13225
+Text GLabel 15625 13225 0    50   Input ~ 0
+Extra4
+Wire Wire Line
+	15625 13325 15700 13325
+Text GLabel 15625 13325 0    50   Input ~ 0
+Extra5
+Wire Wire Line
+	15625 13425 15700 13425
+Text GLabel 15625 13425 0    50   Input ~ 0
+Extra6
+Wire Wire Line
+	15625 13750 15700 13750
+Text GLabel 15625 13750 0    50   Input ~ 0
+Extra8
+Wire Wire Line
+	15625 13850 15700 13850
+Text GLabel 15625 13850 0    50   Input ~ 0
+Extra9
+Wire Wire Line
+	15625 13950 15700 13950
+Text GLabel 15625 13950 0    50   Input ~ 0
+Extra10
+Wire Wire Line
+	15625 14050 15700 14050
+Text GLabel 15625 14050 0    50   Input ~ 0
+Extra11
+Wire Wire Line
+	15625 14150 15700 14150
+Text GLabel 15625 14150 0    50   Input ~ 0
+Extra12
+Wire Wire Line
+	15625 14250 15700 14250
+Text GLabel 15625 14250 0    50   Input ~ 0
+Extra13
+Wire Wire Line
+	15625 14350 15700 14350
+Text GLabel 15625 14350 0    50   Input ~ 0
+Extra14
+Wire Wire Line
+	15625 14450 15700 14450
+Text GLabel 15625 14450 0    50   Input ~ 0
+Extra15
+Wire Wire Line
+	15625 13525 15700 13525
+Text GLabel 15625 13525 0    50   Input ~ 0
+Extra7
+Wire Wire Line
+	21500 15875 21500 15950
+Text GLabel 21500 15875 1    50   Input ~ 0
+Extra1
+Wire Wire Line
+	22175 17600 22100 17600
+Text GLabel 22175 17600 2    50   Input ~ 0
+Extra2
+Wire Wire Line
+	22175 17850 22100 17850
+Text GLabel 22175 17850 2    50   Input ~ 0
+Extra3
+Wire Wire Line
+	22175 18100 22100 18100
+Text GLabel 22175 18100 2    50   Input ~ 0
+Extra4
+Wire Wire Line
+	22175 18350 22100 18350
+Text GLabel 22175 18350 2    50   Input ~ 0
+Extra5
+Wire Wire Line
+	22175 18600 22100 18600
+Text GLabel 22175 18600 2    50   Input ~ 0
+Extra6
+Wire Wire Line
+	22175 18850 22100 18850
+Text GLabel 22175 18850 2    50   Input ~ 0
+Extra7
+Wire Wire Line
+	21250 19475 21250 19400
+Text GLabel 21250 19475 3    50   Input ~ 0
+Extra8
+Wire Wire Line
+	21000 19475 21000 19400
+Text GLabel 21000 19475 3    50   Input ~ 0
+Extra9
+Wire Wire Line
+	20750 19475 20750 19400
+Text GLabel 20750 19475 3    50   Input ~ 0
+Extra10
+Wire Wire Line
+	20500 19475 20500 19400
+Text GLabel 20500 19475 3    50   Input ~ 0
+Extra11
+Wire Wire Line
+	20250 19475 20250 19400
+Text GLabel 20250 19475 3    50   Input ~ 0
+Extra12
+Wire Wire Line
+	20000 19475 20000 19400
+Text GLabel 20000 19475 3    50   Input ~ 0
+Extra13
+Wire Wire Line
+	19750 19475 19750 19400
+Text GLabel 19750 19475 3    50   Input ~ 0
+Extra14
+Wire Wire Line
+	19500 19475 19500 19400
+Text GLabel 19500 19475 3    50   Input ~ 0
+Extra15
+$Comp
+L Mechanical:MountingHole L3
+U 1 1 5D8DFFF3
+P 4725 21575
+F 0 "L3" H 4825 21621 50  0000 L CNN
+F 1 "Keebs Label" H 4825 21530 50  0000 L CNN
+F 2 "keebsLogo:keebsLabel" H 4725 21575 50  0001 C CNN
+F 3 "~" H 4725 21575 50  0001 C CNN
+	1    4725 21575
+	1    0    0    -1
+$EndComp
+$Comp
+L Mechanical:MountingHole L4
+U 1 1 5D8E0395
+P 4725 21825
+F 0 "L4" H 4825 21871 50  0000 L CNN
+F 1 "Keebs Label Mask" H 4825 21780 50  0000 L CNN
+F 2 "keebsLogo:keebsLabelMask" H 4725 21825 50  0001 C CNN
+F 3 "~" H 4725 21825 50  0001 C CNN
+	1    4725 21825
+	1    0    0    -1
+$EndComp

Commit message: Update: README, add renders, add KLE folder
Other:
- note added: "Extra pins"
- note added: "Mounting holes"
- note added: "Switch matrix"
- moved on the sheet: H1, H10, H2, H3, H4, H5, H6, H7, H8, H9, L1, L2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
